Commit message: split function files, modified xml and urdf files

File: robot/arm.urdf (robot description, URDF)
Before this commit: robot arm, 5 links, 4 joints
Links:
- removed link base_link
- added link baselink, mass 2.0; collision box size=0.2 0.2 0.1; visual box size=0.2 0.2 0.1
- added link hand, mass 0.5; collision sphere radius=0.05; visual sphere radius=0.05
- added link shoulder, mass 0.692; collision box size=0.04 0.02 0.24; collision cylinder length=0.032 radius=0.04
- link forearm: geometry collision cylinder length=0.032 radius=0.04; visual box size=0.04 0.02 0.24
- link torso: mass 1.0 -> 0.6684; geometry collision box size=0.06 0.03 0.12; collision cylinder length=0.04 radius=0.06
- link upper_arm: geometry collision cylinder length=0.032 radius=0.04; visual box size=0.04 0.02 0.24
Joints:
- removed joint elbow
- removed joint fixed
- removed joint hip
- removed joint shoulder
- added joint forearm_link: type revolute, parent upper_arm, child forearm, origin xyz=0 0 0.24 rpy=0 0 0, axis 0 -1 0, limit lower=-2.0944 upper=2.0944 effort=10 velocity=2.0
- added joint forearm_to_hand: type fixed, parent forearm, child hand, origin xyz=0 0 0.24 rpy=0 0 0
- added joint shoulder_link: type revolute, parent torso, child shoulder, origin xyz=0 0 0.12 rpy=0 0 0, axis 0 -1 0, limit lower=-2.0944 upper=2.0944 effort=10 velocity=2.0
- added joint torso_bodylink: type revolute, parent baselink, child torso, origin xyz=0 0 0.05 rpy=0 0 0, axis 0 0 1, limit lower=-3.14159 upper=3.14159 effort=10 velocity=2.0
- added joint upper_arm_link: type revolute, parent shoulder, child upper_arm, origin xyz=0 0 0.24 rpy=0 0 0, axis 0 -1 0, limit lower=-2.0944 upper=2.0944 effort=10 velocity=2.0
- added joint world_to_baselink: type fixed, parent world, child baselink, origin xyz=0 0 0.05 rpy=0 0 0

Commit message: modified xml xml and urdf files

File: robot/arm.urdf (robot description, URDF)
Before this commit: robot arm, 7 links, 6 joints
Links:
- link baselink: mass 2.0 -> 4.0; geometry visual box size=0.2 0.2 0.1
- link forearm: geometry visual box size=0.04 0.02 0.24; visual cylinder length=0.032 radius=0.04
- link hand: geometry visual sphere radius=0.05
- link shoulder: mass 0.692 -> 1.0; geometry visual box size=0.04 0.02 0.24; visual cylinder length=0.032 radius=0.04
- link torso: mass 0.6684 -> 0.9; geometry visual box size=0.06 0.03 0.12; visual cylinder length=0.06 radius=0.06
- link upper_arm: geometry visual box size=0.04 0.02 0.24; visual cylinder length=0.032 radius=0.04
Joints:
- joint forearm_link: limit lower=-2.0944 upper=2.0944 effort=10 velocity=2.0 -> lower=-2.1 upper=2.1 effort=10 velocity=2
- joint shoulder_link: limit lower=-2.0944 upper=2.0944 effort=10 velocity=2.0 -> lower=-2.1 upper=2.1 effort=10 velocity=2
- joint torso_bodylink: limit lower=-3.14159 upper=3.14159 effort=10 velocity=2.0 -> lower=-3.14 upper=3.14 effort=10 velocity=2
- joint upper_arm_link: limit lower=-2.0944 upper=2.0944 effort=10 velocity=2.0 -> lower=-2.1 upper=2.1 effort=10 velocity=2

Commit message: updated bot, added hand part, made arm physics better

File: robot/arm.urdf (robot description, URDF)
Before this commit: robot arm, 7 links, 6 joints
Links:
- link baselink: geometry collision box size=0.2 0.2 0.1; visual box size=0.2 0.2 0.1
- link forearm: geometry collision cylinder length=0.032 radius=0.04; visual box size=0.04 0.02 0.24
- link hand: mass 0.5 -> 1.0; geometry collision box size=0.01 0.06 0.1; visual box size=0.01 0.06 0.1
- link shoulder: geometry collision cylinder length=0.032 radius=0.04; visual box size=0.04 0.02 0.24
- link torso: geometry collision box size=0.06 0.03 0.12; collision cylinder length=0.06 radius=0.06
- link upper_arm: geometry collision cylinder length=0.032 radius=0.04; visual box size=0.04 0.02 0.24
Joints:
- removed joint forearm_to_hand
- added joint hand_link: type revolute, parent forearm, child hand, origin xyz=0 0 0.24 rpy=0 0 0, axis 0 0 1, limit lower=-3.14 upper=3.14 effort=100 velocity=10
- joint forearm_link: limit lower=-2.1 upper=2.1 effort=10 velocity=2 -> lower=-2.1 upper=2.1 effort=100 velocity=10
- joint shoulder_link: limit lower=-2.1 upper=2.1 effort=10 velocity=2 -> lower=-2.1 upper=2.1 effort=100 velocity=10
- joint torso_bodylink: limit lower=-3.14 upper=3.14 effort=10 velocity=2 -> lower=-3.14 upper=3.14 effort=100 velocity=10
- joint upper_arm_link: limit lower=-2.1 upper=2.1 effort=10 velocity=2 -> lower=-2.1 upper=2.1 effort=100 velocity=10
